Commit message: done with urdf

File: simulation/src/simple_sim/urdf/eglantyne.xacro (robot description, xacro)
@@ -1,57 +1,30 @@
 <?xml version="1.0"?>
 <robot xmlns:xacro="https://www.ros.org/wiki/xacro" name="eglantyne">
-    <xacro:include filename="body_macro.xacro"/>
-    <link name="world"/>
+    <xacro:include filename="shape_macro.xacro"/>
     <xacro:box_link name="body"
-                    x="80" y="78" z="80"
+                    x="60" y="78" z="80"
                     ofsx="0" ofsy="0" ofsz="40"
-                    mass="1"/>
-    <joint name="fixed" type="fixed">
-        <parent link="world"/>
-        <child link="body"/>
+                    mass="217" collision="true" />
+    <xacro:box_link name="battery"
+                    x="40" y="40" z="80"
+                    ofsx="${-40 / 2}" ofsy="0" ofsz="40"
+                    mass="88" collision="false" />
+    <joint name="battery" type="fixed">
+        <parent link="body"/>
+        <child link="battery"/>
     </joint>
-    <xacro:cylinder_link name="leg_yaw_right"
-                         length="22.2" radious="20"
-                         ofsx="0" ofsy="0" ofsz="-11.1"
-                         mass="1"/>
-    <joint name="leg_yaw_right" type="revolute">
+    <xacro:cylinder_link name="head"
+                         length="50" radius="23"
+                         ofsx="0" ofsy="0" ofsz="${80 + 30 / 2}"
+                         mass="20" collision="true" />
+    <joint name="head" type="fixed">
         <parent link="body"/>
-        <child link="leg_yaw_right"/>
-        <origin xyz="0 0.03 0" rpy="0 0 0"/>
-        <axis xyz="0 0 1"/>
-        <limit lower="-1.57" upper="1.57" effort="10.0" velocity="1.0"/>
+        <child link="head"/>
     </joint>
-    <xacro:box_link name="leg_roll_right"
-                    x="30" y="30" z="26.01"
-                    ofsx="0" ofsy="0" ofsz="${-26.01 / 2}"
-                    mass="1"/>
-    <joint name="leg_roll_right" type="revolute">
-        <parent link="leg_yaw_right"/>
-        <child link="leg_roll_right"/>
-        <origin xyz="0 0 -0.0222" rpy="0 0 0"/>
-        <axis xyz="1 0 0"/>
-        <limit lower="-1.57" upper="1.57" effort="10.0" velocity="1.0"/>
-    </joint>
-    <xacro:box_link name="leg_upper_right"
-                    x="30" y="10" z="78.02"
-                    ofsx="0" ofsy="${10 / 2}" ofsz="${-78.02 / 2}"
-                    mass="1"/>
-    <joint name="leg_upper_right" type="revolute">
-        <parent link="leg_roll_right"/>
-        <child link="leg_upper_right"/>
-        <origin xyz="0 ${0.03 / 2} -0.0261" rpy="0 0 0"/>
-        <axis xyz="0 1 0"/>
-        <limit lower="-1.57" upper="1.57" effort="10.0" velocity="1.0"/>
-    </joint>
-    <xacro:box_link name="leg_under_right"
-                    x="30" y="10" z="78.02"
-                    ofsx="0" ofsy="${-10 / 2}" ofsz="${-78.02 / 2}"
-                    mass="1"/>
-    <joint name="leg_under_right" type="revolute">
-        <parent link="leg_upper_right"/>
-        <child link="leg_under_right"/>
-        <origin xyz="0 0 -0.07802" rpy="0 0 0"/>
-        <axis xyz="0 1 0"/>
-        <limit lower="-1.57" upper="1.57" effort="10.0" velocity="1.0"/>
-    </joint>
+    <xacro:include filename="eglantyne_arm.xacro"/>
+    <xacro:arm_link dir="right"/>
+    <xacro:arm_link dir="left"/>
+    <xacro:include filename="eglantyne_leg.xacro"/>
+    <xacro:leg_link dir="right"/>
+    <xacro:leg_link dir="left"/>
 </robot>

File: simulation/src/simple_sim/urdf/shape_macro.xacro (robot description, xacro)
@@ -1,5 +1,5 @@
 <?xml version="1.0"?>
 <robot xmlns:xacro="https://www.ros.org/wiki/xacro" name="eglantyne">
-    <xacro:macro name="box_link" params="name x y z ofsx ofsy ofsz mass">
+    <xacro:macro name="box_link" params="name x y z ofsx ofsy ofsz mass collision">
         <link name = "${name}">
             <visual>
@@ -12,12 +12,14 @@
                 <origin rpy="0 0 0" xyz="${ofsx * 0.001} ${ofsy * 0.001} ${ofsz * 0.001}"/>
             </visual>
-            <collision>
-                <geometry>
-                    <box size="${x * 0.001} ${y * 0.001} ${z * 0.001}"/>
-                </geometry>
-                <origin rpy="0 0 0" xyz="${ofsx * 0.001} ${ofsy * 0.001} ${ofsz * 0.001}"/>
-            </collision>
+            <xacro:if value="${collision}">
+                <collision>
+                    <geometry>
+                        <box size="${x * 0.001} ${y * 0.001} ${z * 0.001}"/>
+                    </geometry>
+                    <origin rpy="0 0 0" xyz="${ofsx * 0.001} ${ofsy * 0.001} ${ofsz * 0.001}"/>
+                </collision>
+            </xacro:if>
             <inertial>
-                <mass value="${mass}"/>
+                <mass value="${mass * 0.001}"/>
                 <inertia ixx="${(1/12) * mass * (y*y + z*z) * 0.000001}" ixy="0.0" ixz="0.0"
                          iyy="${(1/12) * mass * (x*x + z*z) * 0.000001}" iyz="0.0"
@@ -27,9 +29,9 @@
         </link>
     </xacro:macro>
-    <xacro:macro name="cylinder_link" params="name length radious ofsx ofsy ofsz mass">
+    <xacro:macro name="cylinder_link" params="name length radius ofsx ofsy ofsz mass collision">
         <link name = "${name}">
             <visual>
                 <geometry>
-                    <cylinder length="${length * 0.001}" radius="${radious * 0.001}"/>
+                    <cylinder length="${length * 0.001}" radius="${radius * 0.001}"/>
                 </geometry>
                 <material name="silver">
@@ -38,15 +40,17 @@
                 <origin rpy="0 0 0" xyz="${ofsx * 0.001} ${ofsy * 0.001} ${ofsz * 0.001}"/>
             </visual>
-            <collision>
-                <geometry>
-                    <cylinder length="${length * 0.001}" radius="${radious * 0.001}"/>
-                </geometry>
-                <origin rpy="0 0 0" xyz="${ofsx * 0.001} ${ofsy * 0.001} ${ofsz * 0.001}"/>
-            </collision>
+            <xacro:if value="${collision}">
+                <collision>
+                    <geometry>
+                        <cylinder length="${length * 0.001}" radius="${radius * 0.001}"/>
+                    </geometry>
+                    <origin rpy="0 0 0" xyz="${ofsx * 0.001} ${ofsy * 0.001} ${ofsz * 0.001}"/>
+                </collision>
+            </xacro:if>
             <inertial>
-                <mass value="${mass}"/>
-                <inertia ixx="${( ( (1/4) * mass * radious*radious ) + ( (1/12)* mass * length*length ) )* 0.000001}" ixy="0.0" ixz="0.0"
-                         iyy="${( ( (1/4) * mass * radious*radious ) + ( (1/12)* mass * length*length ) )* 0.000001}" iyz="0.0"
-                         izz="${(1/2) * mass * radious*radious  * 0.000001}" />
+                <mass value="${mass * 0.001}"/>
+                <inertia ixx="${( ( (1/4) * mass * radius*radius ) + ( (1/12)* mass * length*length ) )* 0.000001}" ixy="0.0" ixz="0.0"
+                         iyy="${( ( (1/4) * mass * radius*radius ) + ( (1/12)* mass * length*length ) )* 0.000001}" iyz="0.0"
+                         izz="${(1/2) * mass * radius*radius  * 0.000001}" />
                 <origin rpy="0 0 0" xyz="${ofsx * 0.001} ${ofsy * 0.001} ${ofsz * 0.001}"/>
             </inertial>
