Commit message: add ros2_control

File: simulation/install/simple_sim/share/simple_sim/urdf/body_info/eglantyne_body.xacro (robot description, xacro)
@@ -8,4 +8,5 @@
         <parent link="base"/>
         <child link="body"/>
+        <origin xyz = "0 0 0"/>
     </joint>
     <xacro:box_link name="battery"

File: simulation/install/simple_sim/share/simple_sim/urdf/gazebo_setup.xacro (robot description, xacro)
@@ -2,6 +2,13 @@
 <robot xmlns:xacro="https://www.ros.org/wiki/xacro">
     <gazebo>
+        <plugin name="gazebo_ros2_control" filename="libgazebo_ros2_control.so">
+            <robot_param>robot_description</robot_param>
+            <robot_param_node>robot_state_publisher</robot_param_node>
+            <parameters>$(find simple_sim)/config/eglantyne_controller.yaml</parameters>
+        </plugin>
         <plugin name="gazebo_ros_joint_state_publisher"
             filename="libgazebo_ros_joint_state_publisher.so">
+        <static>false</static>
+        <pose>0 0 0.8 0 0 0</pose>
         <update_rate>20</update_rate>
         <joint_name>arm_pitch_right</joint_name>

File: simulation/install/simple_sim/share/simple_sim/urdf/ros2_control_conf.xacro (robot description, xacro)
@@ -1,77 +1,93 @@
 <?xml version="1.0"?>
 <robot xmlns:xacro="https://www.ros.org/wiki/xacro">
-    <ros2_control name="eglantyne" type="system">
+    <ros2_control name="GazeboSystem" type="system">
         <hardware>
             <plugin>gazebo_ros2_control/GazeboSystem</plugin>
         </hardware>
-        <xacro:macro name="ros2_control_joint" params="name posmin posmax angle_init">
-            <joint name="${name}">
-                <command_interface name="position">
-                    <param name="min">${posmin}</param>
-                    <param name="max">${posmin}</param>
-                </command_interface>
-                <command_interface name="velocity">
-                    <param name="min">-3.15</param>
-                    <param name="max">3.15</param>
-                </command_interface>
-                <state_interface name="position">
-                    <param name="initial_value">${angle_init}</param>
-                </state_interface>
-            </joint>
+        <xacro:macro name="ros2_control_joint" params="posmin posmax angle_init">
+            <command_interface name="position">
+                <param name="min">${posmin}</param>
+                <param name="max">${posmin}</param>
+            </command_interface>
+            <command_interface name="velocity">
+                <param name="min">-3.15</param>
+                <param name="max">3.15</param>
+            </command_interface>
+            <state_interface name="position">
+                <param name="initial_value">${angle_init}</param>
+            </state_interface>
         </xacro:macro>
-        <xacro:ros2_control_joint name = "arm_pitch_right"
-                                  posmin="-3.14" posmax="1.57"
-                                  angle_init="${-3.14 / 2}" />
-        <xacro:ros2_control_joint name = "arm_roll_right"
-                                  posmin="${-3.14 * 7 / 6}" posmax="${3.14 / 6}"
-                                  angle_init="0" />
-        <xacro:ros2_control_joint name = "hand_right"
-                                  posmin="-3.14" posmax="${3.14 / 4}"
-                                  angle_init="-1.57" />
-        <xacro:ros2_control_joint name = "arm_pitch_left"
-                                  posmin="-1.57" posmax="3.14"
-                                  angle_init="${3.14 / 4}" />
-        <xacro:ros2_control_joint name = "arm_roll_left"
-                                  posmin="${-3.14 / 6}" posmax="${3.14 * 7 / 6}"
-                                  angle_init="0" />
-        <xacro:ros2_control_joint name = "hand_left"
-                                  posmin="-3.14" posmax="${3.14 / 4}"
-                                  angle_init="-1.57" />
-        <xacro:ros2_control_joint name = "leg_yaw_right"
-                                  posmin="-1.57" posmax="1.57"
-                                  angle_init="0" />
-        <xacro:ros2_control_joint name = "leg_roll_right"
-                                  posmin="-1.57" posmax="${3.14 / 6}"
-                                  angle_init="0" />
-        <xacro:ros2_control_joint name = "leg_upper_right"
-                                  posmin="${-3.14 * 5 / 6}" posmax="${3.14 / 4}"
-                                  angle_init="${-3.14 / 6}" />
-        <xacro:ros2_control_joint name = "leg_under_right"
-                                  posmin="0" posmax="${3.14 * 5 / 6}"
-                                  angle_init="${3.14 / 3}" />
-        <xacro:ros2_control_joint name = "foot_pitch_right"
-                                  posmin="${-3.14 / 3}" posmax="0"
-                                  angle_init="${-3.14 / 6}" />
-        <xacro:ros2_control_joint name = "foot_roll_right"
-                                  posmin="${-3.14 / 3}" posmax="${3.14 / 3}"
-                                  angle_init="0" />
-        <xacro:ros2_control_joint name = "leg_yaw_left"
-                                  posmin="-1.57" posmax="1.57"
-                                  angle_init="0" />
-        <xacro:ros2_control_joint name = "leg_roll_left"
-                                  posmin="${3.14 / 6}" posmax="1.57"
-                                  angle_init="0" />
-        <xacro:ros2_control_joint name = "leg_upper_left"
-                                  posmin="${-3.14 * 5 / 6}" posmax="${3.14 / 4}"
-                                  angle_init="${-3.14 / 6}" />
-        <xacro:ros2_control_joint name = "leg_under_left"
-                                  posmin="0" posmax="${3.14 * 5 / 6}"
-                                  angle_init="${3.14 / 3}" />
-        <xacro:ros2_control_joint name = "foot_pitch_left"
-                                  posmin="${-3.14 / 3}" posmax="0"
-                                  angle_init="${-3.14 / 6}" />
-        <xacro:ros2_control_joint name = "foot_roll_left"
-                                  posmin="${-3.14 / 3}" posmax="${3.14 / 3}"
-                                  angle_init="0" />
+        <joint name = "arm_pitch_right">
+            <xacro:ros2_control_joint  posmin="-3.14" posmax="1.57"
+                                       angle_init="0" />
+        </joint>
+        <joint name = "arm_roll_right">
+            <xacro:ros2_control_joint  posmin="${-3.14 * 7 / 6}" posmax="${3.14 / 6}"
+                                       angle_init="0" />
+        </joint>
+        <joint name = "hand_right">
+            <xacro:ros2_control_joint  posmin="-3.14" posmax="${3.14 / 4}"
+                                       angle_init="${-3.14 / 4}" />
+        </joint>
+        <joint name = "arm_pitch_left">
+            <xacro:ros2_control_joint  posmin="-1.57" posmax="3.14"
+                                       angle_init="0" />
+        </joint>
+        <joint name = "arm_roll_left">
+            <xacro:ros2_control_joint  posmin="${-3.14 / 6}" posmax="${3.14 * 7 / 6}"
+                                       angle_init="0" />
+        </joint>
+        <joint name = "hand_left">
+            <xacro:ros2_control_joint  posmin="-3.14" posmax="${3.14 / 4}"
+                                       angle_init="${-3.14 / 4}" />
+        </joint>
+        <joint name = "leg_yaw_right">
+            <xacro:ros2_control_joint  posmin="-1.57" posmax="1.57"
+                                       angle_init="0" />
+        </joint>
+        <joint name = "leg_roll_right">
+            <xacro:ros2_control_joint  posmin="-1.57" posmax="${3.14 / 6}"
+                                       angle_init="0" />
+        </joint>
+        <joint name = "leg_upper_right">
+            <xacro:ros2_control_joint  posmin="${-3.14 * 5 / 6}" posmax="${3.14 / 4}"
+                                       angle_init="${-3.14 / 6}" />
+        </joint>
+        <joint name = "leg_under_right">
+            <xacro:ros2_control_joint  posmin="0" posmax="${3.14 * 5 / 6}"
+                                       angle_init="${3.14 / 3}" />
+        </joint>
+        <joint name = "foot_pitch_right">
+            <xacro:ros2_control_joint  posmin="${-3.14 / 3}" posmax="0"
+                                       angle_init="${-3.14 / 6}" />
+        </joint>
+        <joint name = "foot_roll_right">
+            <xacro:ros2_control_joint  posmin="${-3.14 / 3}" posmax="${3.14 / 3}"
+                                       angle_init="0" />
+        </joint>
+        <joint name = "leg_yaw_left">
+            <xacro:ros2_control_joint  posmin="-1.57" posmax="1.57"
+                                       angle_init="0" />
+        </joint>
+        <joint name = "leg_roll_left">
+            <xacro:ros2_control_joint  posmin="${3.14 / 6}" posmax="1.57"
+                                       angle_init="0" />
+        </joint>
+        <joint name = "leg_upper_left">
+            <xacro:ros2_control_joint  posmin="${-3.14 * 5 / 6}" posmax="${3.14 / 4}"
+                                       angle_init="${-3.14 / 6}" />
+        </joint>
+        <joint name = "leg_under_left">
+            <xacro:ros2_control_joint  posmin="0" posmax="${3.14 * 5 / 6}"
+                                       angle_init="${3.14 / 3}" />
+        </joint>
+        <joint name = "foot_pitch_left">
+            <xacro:ros2_control_joint  posmin="${-3.14 / 3}" posmax="0"
+                                       angle_init="${-3.14 / 6}" />
+        </joint>
+        <joint name = "foot_roll_left">
+            <xacro:ros2_control_joint  posmin="${-3.14 / 3}" posmax="${3.14 / 3}"
+                                       angle_init="0" />
+        </joint>
     </ros2_control>
 </robot>

Commit message: move simulation

File: simulation/install/simple_sim/share/simple_sim/urdf/body_info/eglantyne_body.xacro (robot description, xacro)
@@ -6,7 +6,6 @@
                     mass="217" collision="true" />
     <joint name="fixed" type="fixed">
-        <parent link="base"/>
-        <child link="body"/>
-        <origin xyz = "0 0 0"/>
+        <parent link="base_link"/>
+        <child link="body_link"/>
     </joint>
     <xacro:box_link name="battery"
@@ -15,6 +14,6 @@
                     mass="88" collision="false" />
     <joint name="battery" type="fixed">
-        <parent link="body"/>
-        <child link="battery"/>
+        <parent link="body_link"/>
+        <child link="battery_link"/>
     </joint>
     <xacro:cylinder_link name="head"
@@ -23,6 +22,6 @@
                          mass="20" collision="true" />
     <joint name="head" type="fixed">
-        <parent link="body"/>
-        <child link="head"/>
+        <parent link="body_link"/>
+        <child link="head_link"/>
     </joint>
 </robot>

File: simulation/install/simple_sim/share/simple_sim/urdf/body_info/shape_macro.xacro (robot description, xacro)
@@ -2,5 +2,5 @@
 <robot xmlns:xacro="https://www.ros.org/wiki/xacro" name="eglantyne">
     <xacro:macro name="box_link" params="name x y z ofsx ofsy ofsz mass collision">
-        <link name = "${name}">
+        <link name = "${name}_link">
             <visual>
                 <geometry>
@@ -30,5 +30,5 @@
     </xacro:macro>
     <xacro:macro name="cylinder_link" params="name length radius ofsx ofsy ofsz mass collision">
-        <link name = "${name}">
+        <link name = "${name}_link">
             <visual>
                 <geometry>

File: simulation/install/simple_sim/share/simple_sim/urdf/eglantyne.xacro (robot description, xacro)
@@ -2,14 +2,12 @@
 <robot xmlns:xacro="https://www.ros.org/wiki/xacro" name="eglantyne">
     <xacro:include filename="body_info/shape_macro.xacro"/>
-    <link name="base"/>
+    <link name="base_link"/>
     <xacro:include filename="body_info/eglantyne_body.xacro"/>
-    <xacro:include filename="body_info/eglantyne_arm_right.xacro"/>
-    <xacro:arm_right_link dir="right"/>
-    <xacro:include filename="body_info/eglantyne_arm_left.xacro"/>
-    <xacro:arm_left_link dir="left"/>
-    <xacro:include filename="body_info/eglantyne_leg_right.xacro"/>
-    <xacro:leg_right_link dir="right"/>
-    <xacro:include filename="body_info/eglantyne_leg_left.xacro"/>
-    <xacro:leg_left_link dir="left"/>
+    <xacro:include filename="body_info/eglantyne_arm.xacro"/>
+    <xacro:arm_link dir="right"/>
+    <xacro:arm_link dir="left"/>
+    <xacro:include filename="body_info/eglantyne_leg.xacro"/>
+    <xacro:leg_link dir="right"/>
+    <xacro:leg_link dir="left"/>
     <xacro:include filename="gazebo_setup.xacro"/>
     <xacro:include filename="ros2_control_conf.xacro"/>

File: simulation/install/simple_sim/share/simple_sim/urdf/gazebo_setup.xacro (robot description, xacro)
@@ -9,6 +9,4 @@
         <plugin name="gazebo_ros_joint_state_publisher"
             filename="libgazebo_ros_joint_state_publisher.so">
-        <static>false</static>
-        <pose>0 0 0.8 0 0 0</pose>
         <update_rate>20</update_rate>
         <joint_name>arm_pitch_right</joint_name>

File: simulation/install/simple_sim/share/simple_sim/urdf/ros2_control_conf.xacro (robot description, xacro)
@@ -5,89 +5,73 @@
             <plugin>gazebo_ros2_control/GazeboSystem</plugin>
         </hardware>
-        <xacro:macro name="ros2_control_joint" params="posmin posmax angle_init">
-            <command_interface name="position">
-                <param name="min">${posmin}</param>
-                <param name="max">${posmin}</param>
-            </command_interface>
-            <command_interface name="velocity">
-                <param name="min">-3.15</param>
-                <param name="max">3.15</param>
-            </command_interface>
-            <state_interface name="position">
-                <param name="initial_value">${angle_init}</param>
-            </state_interface>
+        <xacro:macro name="ros2_control_joint" params="name posmin posmax angle_init">
+            <joint name="${name}">
+                <command_interface name="position">
+                    <param name="min">${posmin}</param>
+                    <param name="max">${posmin}</param>
+                </command_interface>
+                <command_interface name="velocity">
+                    <param name="min">-3.15</param>
+                    <param name="max">3.15</param>
+                </command_interface>
+                <state_interface name="position">
+                    <param name="initial_value">${angle_init}</param>
+                </state_interface>
+            </joint>
         </xacro:macro>
-        <joint name = "arm_pitch_right">
-            <xacro:ros2_control_joint  posmin="-3.14" posmax="1.57"
-                                       angle_init="0" />
-        </joint>
-        <joint name = "arm_roll_right">
-            <xacro:ros2_control_joint  posmin="${-3.14 * 7 / 6}" posmax="${3.14 / 6}"
-                                       angle_init="0" />
-        </joint>
-        <joint name = "hand_right">
-            <xacro:ros2_control_joint  posmin="-3.14" posmax="${3.14 / 4}"
-                                       angle_init="${-3.14 / 4}" />
-        </joint>
-        <joint name = "arm_pitch_left">
-            <xacro:ros2_control_joint  posmin="-1.57" posmax="3.14"
-                                       angle_init="0" />
-        </joint>
-        <joint name = "arm_roll_left">
-            <xacro:ros2_control_joint  posmin="${-3.14 / 6}" posmax="${3.14 * 7 / 6}"
-                                       angle_init="0" />
-        </joint>
-        <joint name = "hand_left">
-            <xacro:ros2_control_joint  posmin="-3.14" posmax="${3.14 / 4}"
-                                       angle_init="${-3.14 / 4}" />
-        </joint>
-        <joint name = "leg_yaw_right">
-            <xacro:ros2_control_joint  posmin="-1.57" posmax="1.57"
-                                       angle_init="0" />
-        </joint>
-        <joint name = "leg_roll_right">
-            <xacro:ros2_control_joint  posmin="-1.57" posmax="${3.14 / 6}"
-                                       angle_init="0" />
-        </joint>
-        <joint name = "leg_upper_right">
-            <xacro:ros2_control_joint  posmin="${-3.14 * 5 / 6}" posmax="${3.14 / 4}"
-                                       angle_init="${-3.14 / 6}" />
-        </joint>
-        <joint name = "leg_under_right">
-            <xacro:ros2_control_joint  posmin="0" posmax="${3.14 * 5 / 6}"
-                                       angle_init="${3.14 / 3}" />
-        </joint>
-        <joint name = "foot_pitch_right">
-            <xacro:ros2_control_joint  posmin="${-3.14 / 3}" posmax="0"
-                                       angle_init="${-3.14 / 6}" />
-        </joint>
-        <joint name = "foot_roll_right">
-            <xacro:ros2_control_joint  posmin="${-3.14 / 3}" posmax="${3.14 / 3}"
-                                       angle_init="0" />
-        </joint>
-        <joint name = "leg_yaw_left">
-            <xacro:ros2_control_joint  posmin="-1.57" posmax="1.57"
-                                       angle_init="0" />
-        </joint>
-        <joint name = "leg_roll_left">
-            <xacro:ros2_control_joint  posmin="${3.14 / 6}" posmax="1.57"
-                                       angle_init="0" />
-        </joint>
-        <joint name = "leg_upper_left">
-            <xacro:ros2_control_joint  posmin="${-3.14 * 5 / 6}" posmax="${3.14 / 4}"
-                                       angle_init="${-3.14 / 6}" />
-        </joint>
-        <joint name = "leg_under_left">
-            <xacro:ros2_control_joint  posmin="0" posmax="${3.14 * 5 / 6}"
-                                       angle_init="${3.14 / 3}" />
-        </joint>
-        <joint name = "foot_pitch_left">
-            <xacro:ros2_control_joint  posmin="${-3.14 / 3}" posmax="0"
-                                       angle_init="${-3.14 / 6}" />
-        </joint>
-        <joint name = "foot_roll_left">
-            <xacro:ros2_control_joint  posmin="${-3.14 / 3}" posmax="${3.14 / 3}"
-                                       angle_init="0" />
-        </joint>
-    </ros2_control>
+        <xacro:ros2_control_joint  name = "arm_pitch_right"
+                                   posmin="-3.14" posmax="1.57"
+                                   angle_init="0" />
+        <xacro:ros2_control_joint  name = "arm_roll_right"
+                                   posmin="${-3.14 * 7 / 6}" posmax="${3.14 / 6}"
+                                   angle_init="0" />
+        <xacro:ros2_control_joint  name = "hand_right"
+                                   posmin="-3.14" posmax="${3.14 / 4}"
+                                   angle_init="${-3.14 / 4}" />
+        <xacro:ros2_control_joint  name = "arm_pitch_left"
+                                   posmin="-1.57" posmax="3.14"
+                                   angle_init="0" />
+        <xacro:ros2_control_joint  name = "arm_roll_left"
+                                   posmin="${-3.14 / 6}" posmax="${3.14 * 7 / 6}"
+                                   angle_init="0" />
+        <xacro:ros2_control_joint  name = "hand_left"
+                                   posmin="-3.14" posmax="${3.14 / 4}"
+                                   angle_init="${-3.14 / 4}" />
+        <xacro:ros2_control_joint  name = "leg_yaw_right"
+                                   posmin="-1.57" posmax="1.57"
+                                   angle_init="0" />
+        <xacro:ros2_control_joint  name = "leg_roll_right"
+                                   posmin="-1.57" posmax="${3.14 / 6}"
+                                   angle_init="0" />
+        <xacro:ros2_control_joint  name = "leg_upper_right"
+                                   posmin="${-3.14 * 5 / 6}" posmax="${3.14 / 4}"
+                                   angle_init="${-3.14 / 6}" />
+        <xacro:ros2_control_joint  name = "leg_under_right"
+                                   posmin="0" posmax="${3.14 * 5 / 6}"
+                                   angle_init="${3.14 / 3}" />
+        <xacro:ros2_control_joint  name = "foot_pitch_right"
+                                   posmin="${-3.14 / 3}" posmax="0"
+                                   angle_init="${-3.14 / 6}" />
+        <xacro:ros2_control_joint  name = "foot_roll_right"
+                                   posmin="${-3.14 / 3}" posmax="${3.14 / 3}"
+                                   angle_init="0" />
+        <xacro:ros2_control_joint  name = "leg_yaw_left"
+                                   posmin="-1.57" posmax="1.57"
+                                   angle_init="0" />
+        <xacro:ros2_control_joint  name = "leg_roll_left"
+                                   posmin="${3.14 / 6}" posmax="1.57"
+                                   angle_init="0" />
+        <xacro:ros2_control_joint  name = "leg_upper_left"
+                                   posmin="${-3.14 * 5 / 6}" posmax="${3.14 / 4}"
+                                   angle_init="${-3.14 / 6}" />
+        <xacro:ros2_control_joint  name = "leg_under_left"
+                                   posmin="0" posmax="${3.14 * 5 / 6}"
+                                   angle_init="${3.14 / 3}" />
+        <xacro:ros2_control_joint  name = "foot_pitch_left"
+                                   posmin="${-3.14 / 3}" posmax="0"
+                                   angle_init="${-3.14 / 6}" />
+        <xacro:ros2_control_joint  name = "foot_roll_left"
+                                   posmin="${-3.14 / 3}" posmax="${3.14 / 3}"
+                                   angle_init="0" />
+   </ros2_control>
 </robot>
