Commit message: change control method to effort control

File: simulation/install/simple_sim/share/simple_sim/urdf/body_info/eglantyne_arm.xacro (robot description, xacro)
@@ -16,8 +16,8 @@
         <axis xyz="0 0 1"/>
         <xacro:if value="${dir == 'right'}">
-            <limit lower="-3.14" upper="1.57" effort="10.0" velocity="1.0"/>
+            <limit lower="-3.14" upper="1.57" effort="25" velocity="6.8"/>
         </xacro:if>
         <xacro:if value="${dir == 'left'}">
-            <limit lower="-1.57" upper="3.14" effort="10.0" velocity="1.0"/>
+            <limit lower="-1.57" upper="3.14" effort="25" velocity="6.8"/>
         </xacro:if>
     </joint>
@@ -37,8 +37,8 @@
         <axis xyz="1 0 0"/>
         <xacro:if value="${dir == 'right'}">
-            <limit lower="${-3.14 * 7 / 6}" upper="${3.14 / 6}" effort="10.0" velocity="1.0"/>
+            <limit lower="${-3.14 * 7 / 6}" upper="${3.14 / 6}" effort="25" velocity="6.8"/>
         </xacro:if>
         <xacro:if value="${dir == 'left'}">
-            <limit lower="${-3.14 / 6}" upper="${3.14 * 7 / 6}" effort="10.0" velocity="1.0"/>
+            <limit lower="${-3.14 / 6}" upper="${3.14 * 7 / 6}" effort="25" velocity="6.8"/>
         </xacro:if>
     </joint>
@@ -52,5 +52,5 @@
         <origin xyz="0 0 -0.08284" rpy="0 0 0"/>
         <axis xyz="0 1 0"/>
-        <limit lower="-3.14" upper="${3.14 / 4}" effort="10.0" velocity="1.0"/>
+        <limit lower="-3.14" upper="${3.14 / 4}" effort="25" velocity="6.8"/>
     </joint>
 </xacro:macro>

File: simulation/install/simple_sim/share/simple_sim/urdf/body_info/eglantyne_leg.xacro (robot description, xacro)
@@ -15,5 +15,5 @@
         </xacro:if>
         <axis xyz="0 0 1"/>
-        <limit lower="-1.57" upper="1.57" effort="10.0" velocity="1.0"/>
+        <limit lower="-1.57" upper="1.57" effort="25" velocity="6.8"/>
     </joint>
     <xacro:box_link name="leg_roll_${dir}"
@@ -27,8 +27,8 @@
         <axis xyz="1 0 0"/>
         <xacro:if value="${dir == 'right'}">
-            <limit lower="-1.57" upper="${3.14 / 6}" effort="10.0" velocity="1.0"/>
+            <limit lower="-1.57" upper="${3.14 / 6}" effort="25" velocity="6.8"/>
         </xacro:if>
         <xacro:if value="${dir == 'left'}">
-            <limit lower="${-3.14 / 6}" upper="1.57" effort="10.0" velocity="1.0"/>
+            <limit lower="${-3.14 / 6}" upper="1.57" effort="25" velocity="6.8"/>
         </xacro:if>
     </joint>
@@ -42,5 +42,5 @@
         <origin xyz="0 0 -0.0261" rpy="0 0 0"/>
         <axis xyz="0 1 0"/>
-        <limit lower="${-3.14 * 5 / 6}" upper="${3.14 / 4}" effort="10.0" velocity="1.0"/>
+        <limit lower="${-3.14 * 5 / 6}" upper="${3.14 / 4}" effort="25" velocity="6.8"/>
     </joint>
     <xacro:box_link name="leg_under_${dir}"
@@ -53,5 +53,5 @@
         <origin xyz="0 0 -0.07802" rpy="0 0 0"/>
         <axis xyz="0 1 0"/>
-        <limit lower="0" upper="${3.14 * 5 / 6}" effort="10.0" velocity="1.0"/>
+        <limit lower="0" upper="${3.14 * 5 / 6}" effort="25" velocity="6.8"/>
     </joint>
     <xacro:cylinder_link name="foot_pitch_${dir}"
@@ -64,5 +64,5 @@
         <origin xyz="0 0 -0.07802" rpy="0 -1.57 0"/>
         <axis xyz="0 1 0"/>
-        <limit lower="${-3.14 / 3}" upper="0" effort="10.0" velocity="1.0"/>
+        <limit lower="${-3.14 / 3}" upper="0" effort="25" velocity="6.8"/>
     </joint>
     <xacro:cylinder_link name="foot_roll_${dir}"
@@ -75,5 +75,5 @@
         <origin xyz="0 0 -0.03" rpy="0 0 0"/>
         <axis xyz="0 0 1"/>
-        <limit lower="${-3.14 / 3}" upper="${3.14 / 3}" effort="10.0" velocity="1.0"/>
+        <limit lower="${-3.14 / 3}" upper="${3.14 / 3}" effort="25" velocity="6.8"/>
     </joint>
     <xacro:box_link name="foot_${dir}"

File: simulation/install/simple_sim/share/simple_sim/urdf/body_info/shape_macro.xacro (robot description, xacro)
@@ -1,4 +1,21 @@
 <?xml version="1.0"?>
 <robot xmlns:xacro="https://www.ros.org/wiki/xacro" name="eglantyne">
+    <xacro:macro name="surface">
+        <surcafe>
+            <friction>
+                <ode>
+                    <mu1>50</mu1>
+                    <mu2>25</mu2>
+                </ode>
+            </friction>
+            <contact>
+                <ode>
+                    <kp>25000</kp>
+                    <kd>0.05</kd>
+                    <damping_factor>0.004</damping_factor>
+                </ode>
+            </contact>
+        </surcafe>
+    </xacro:macro>
     <xacro:macro name="box_link" params="name x y z ofsx ofsy ofsz mass collision">
         <link name = "${name}_link">
@@ -27,4 +44,5 @@
                 <origin rpy="0 0 0" xyz="${ofsx * 0.001} ${ofsy * 0.001} ${ofsz * 0.001}"/>
             </inertial>
+            <xacro:macro name="surcafe"/>
         </link>
     </xacro:macro>
@@ -55,4 +73,5 @@
                 <origin rpy="0 0 0" xyz="${ofsx * 0.001} ${ofsy * 0.001} ${ofsz * 0.001}"/>
             </inertial>
+            <xacro:macro name="surcafe"/>
         </link>
     </xacro:macro>

File: simulation/install/simple_sim/share/simple_sim/urdf/ros2_control_conf.xacro (robot description, xacro)
@@ -11,12 +11,10 @@
                     <param name="max">${posmin}</param>
                 </command_interface>
-                <command_interface name="velocity">
-                    <param name="min">-3.15</param>
-                    <param name="max">3.15</param>
-                </command_interface>
+                <command_interface name="velocity"/>
+                <command_interface name="effort"/>
                 <state_interface name="position">
                     <param name="initial_value">${angle_init}</param>
                 </state_interface>
-                <state_interface name="velocity"/>
+                <state_interface name="velocity"/>]
                 <!-- <state_interface name="effort"/> -->
             </joint>
@@ -48,13 +46,13 @@
         <xacro:ros2_control_joint  name = "leg_upper_right"
                                    posmin="${-3.14 * 5 / 6}" posmax="${3.14 / 4}"
-                                   angle_init="${-3.14 / 6}" />
+                                   angle_init="${-3.14 * 18.31 / 180}" />
         <xacro:ros2_control_joint  name = "leg_under_right"
                                    posmin="0" posmax="${3.14 * 5 / 6}"
-                                   angle_init="${3.14 / 3}" />
+                                   angle_init="${3.14 * 65.8 / 180}" />
         <xacro:ros2_control_joint  name = "foot_pitch_right"
                                    posmin="${-3.14 / 3}" posmax="0"
-                                   angle_init="${-3.14 / 6}" />
+                                   angle_init="${-3.14 * 45.88 / 180}" />
         <xacro:ros2_control_joint  name = "foot_roll_right"
-                                   posmin="${-3.14 / 3}" posmax="${3.14 / 3}"
+                                   posmin="${-3.14 /3}" posmax="${3.14 / 3}"
                                    angle_init="0" />
         <xacro:ros2_control_joint  name = "leg_yaw_left"
@@ -66,13 +64,13 @@
         <xacro:ros2_control_joint  name = "leg_upper_left"
                                    posmin="${-3.14 * 5 / 6}" posmax="${3.14 / 4}"
-                                   angle_init="${-3.14 / 6}" />
+                                   angle_init="${-3.14 * 18.31 / 180}" />
         <xacro:ros2_control_joint  name = "leg_under_left"
                                    posmin="0" posmax="${3.14 * 5 / 6}"
-                                   angle_init="${3.14 / 3}" />
+                                   angle_init="${3.14 * 65.8 / 180}" />
         <xacro:ros2_control_joint  name = "foot_pitch_left"
                                    posmin="${-3.14 / 3}" posmax="0"
-                                   angle_init="${-3.14 / 6}" />
+                                   angle_init="${-3.14 * 45.88 / 180}" />
         <xacro:ros2_control_joint  name = "foot_roll_left"
-                                   posmin="${-3.14 / 3}" posmax="${3.14 / 3}"
+                                   posmin="${-3.14 /3}" posmax="${3.14 / 3}"
                                    angle_init="0" />
    </ros2_control>
